File: Schematic/UPL_B1/Sheet2.kicad_sch (KiCad schematic)
At the start: 0 parts

Commit message: added connections and library
Other:
- company: (none) -> BVKSound
- title: (none) -> UPL-B1: OUTPUT IMD ATTENUATOR
Changed lines of the file:
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@@
 	(generator_version "9.0")
 	(paper "A4")
+	(title_block
+		(title "UPL-B1: OUTPUT IMD ATTENUATOR")
+		(date "2025-11-24")
+		(rev "1.0")
+		(company "BVKSound")
+	)
 )
