File: Schematic/UPL_B1/Sheet6.kicad_sch (KiCad schematic)
At the start: 0 parts

Commit message: added connections and library
Parts:
- added X1: 5102159-8, TYCO_5102159-8, symbol UPL_B1:5102159-8
- added X3, X4: Conn_01x06_Pin, symbol Connector:Conn_01x06_Pin
Connections:
- new net +15V: X1.19, X1.20, X4.2 (Pin_2)
- new net +5V: X1.23, X1.24, X4.1 (Pin_1)
- new net +6V: X1.21, X1.22, X4.5 (Pin_5)
- new net -15V: X1.17, X1.18, X4.3 (Pin_3)
- new net -24V: X1.15, X1.16, X4.4 (Pin_4)
- new net -5V: X1.14
- new net CLK: X1.12, X3.4 (Pin_4)
- new net ENABLE: X1.7, X4.6 (Pin_6)
- new net GNDD: X1.1, X1.13, X1.25, X1.26, X1.27, X1.28, X1.29, X1.3, X1.30, X1.31, X1.32, X1.33, X1.4, X1.5, X1.6
- new net LDFRQ: X1.2
- new net LOW DIST: X1.34
- new net SDI: X1.11, X3.5 (Pin_5)
- new net SDO: X1.8, X3.6 (Pin_6)
- new net WR: X3.1 (Pin_1)
- new net ~{RD}: X1.10, X3.3 (Pin_3)
- new net ~{WR}: X1.9, X3.2 (Pin_2)
Other:
- note added: "2"
- note added: "2/3/4"
- note added: "2/3/4/5"
- note added: "3"
- note added: "5/6"
- note added: "SHEET"
- company: (none) -> BVKSound
- title: (none) -> UPL-B1: Connections
Changed lines of the file:
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@@
 	(generator_version "9.0")
 	(paper "A4")
-)
+	(title_block
+		(title "UPL-B1: Connections")
+		(date "2025-11-24")
+		(rev "1.0")
+		(company "BVKSound")
+	)
