File: Schematic/UPL_B1/UPL_B1.kicad_sch (KiCad schematic)
At the start: 0 parts

Commit message: Connections page added
Other:
- added sheet Connections (Sheet6.kicad_sch)

Commit message: added connections and library
Other:
- company: (none) -> BVKSound
- title: (none) -> UPL-B1: Block Diagram
Changed lines of the file:
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@@
 	(generator_version "9.0")
 	(paper "A2")
+	(title_block
+		(title "UPL-B1: Block Diagram")
+		(date "2025-11-24")
+		(rev "1.0")
+		(company "BVKSound")
+	)
 	(image
 		(at 298.45 139.7)
