File: Schematic/UPL_B1/Sheet4.kicad_sch (KiCad schematic)
At the start: 0 parts

Commit message: added connections and library
Other:
- company: (none) -> BVKSound
- title: (none) -> UPL-B1: Integrator 2
Changed lines of the file:
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@@
 	(generator_version "9.0")
 	(paper "A4")
+	(title_block
+		(title "UPL-B1: Integrator 2")
+		(date "2025-11-24")
+		(rev "1.0")
+		(company "BVKSound")
+	)
 )

Commit message: Integrator 2 schematic added
Parts:
- added C2: 2n2 100V 1% FKP, symbol Device:C_Small
- added C400, C401: 3P9, symbol Device:C_Small
- added C402: 330nF, symbol Device:C_Small
- added C404: 33n 63V 1% FKP, symbol Device:C_Small
- added C405: 560p, symbol Device:C_Small
- added C406, C407, C408, C409, C410: 100nF, symbol Device:C_Small
- added C414: 220uF 35V, symbol Device:C_Polarized_Small
- added C415: 330pF, symbol Device:C_Small
- added D40: DAC8143FSZ, SOIC127P1032X265-16N, symbol UPL_B1:DAC8143FSZ
- added D41: 74HCT4094D,118, 74HCT4094D118, symbol UPL_B1:74HCT4094D,118
- added N40: NE5534 / SE5534, symbol Amplifier_Operational:NE5534
- added N41: LM339, symbol Comparator:LM339
- added N42: HA7-5221, Package_SO:MSOP-8_3x3mm_P0.65mm, symbol Amplifier_Operational:OP1177ARM
- added R400: 5K05 0.1%, symbol Device:R_Small
- added R401: 511K, symbol Device:R_Small
- added R402: 10K 0.1%, symbol Device:R_Small
- added R403: 20K 0.1%, symbol Device:R_Small
- added R404: 38K8 0.1%, symbol Device:R_Small
- added R405: 1K21, symbol Device:R_Small
- added R406, R408: 41K7 0.1%, symbol Device:R_Small
- added R407, R409: 1M, symbol Device:R_Small
- added R410, R411, R420: 1K, symbol Device:R_Small
- added R412, R413, R414, R415, R416, R417, R418, R419: 15K, symbol Device:R_Small
- added R421, R422, R423, R424, R425, R426: 100K, symbol Device:R_Small
- added R427, R428, R429: 10K, symbol Device:R_Small
- added R430: 100R, symbol Device:R_Small
- added V400, V401, V402, V403: BC860B, symbol Transistor_BJT:Q_PNP_BCE
- added V404: J105, symbol Simulation_SPICE:NJFET
- added V405: SST108, symbol Simulation_SPICE:NJFET
- added V406, V407: BSR56, symbol Simulation_SPICE:NJFET
- added V408, V409, V410: 2N5432, symbol Simulation_SPICE:NJFET
Connections:
- new net: C404.2, R424.2, R428.1, V409.3 (S)
- new net: D40.10 (~{STB3}), D40.13 (~{CLR}), R410.2
- new net: R404.2, V403.2 (C), V407.1 (D)
- new net: N41.2, R415.2, R419.1, V407.2 (G)
- new net: C405.2, N42.2 (-), R406.2, R407.2, R408.1, R409.1, V404.1 (D), V405.1 (D), V406.1 (D), V407.3 (S), V408.1 (D), V409.1 (D), V410.1 (D)
- new net: C402.2, R422.2, R427.1, V408.3 (S)
- new net: D41.15 (OE), R420.2
- new net: D40.6 (SRO), D41.2 (D)
- new net: D41.4 (QP0), N41.4 (-)
- new net: D41.5 (QP1), N41.6 (-)
- new net: D41.6 (QP2), N41.8 (-)
- new net: D41.7 (QP3), N41.10 (-)
- new net: N41.13, R412.2, R416.1, V404.2 (G)
- new net: R415.1, V403.1 (B)
- new net: R412.1, V400.1 (B)
- new net: R400.2, R401.2, V400.2 (C), V404.3 (S)
- new net: R403.2, V402.2 (C), V406.3 (S)
- new net: C400.2, D40.1 (IOUT1), N40.2 (-), N40.6, R408.2, R409.2
- new net: C2.2, R426.2, R429.1, V410.3 (S)
- new net: D40.11 (STB4), D40.4 (STB1), D40.5 (~{LD1}), R411.1
- new net: C400.1, D40.16 (RFB)
- new net: R413.1, V401.1 (B)
- new net: N41.14, R413.2, R417.1, V405.2 (G)
- new net: R414.1, V402.1 (B)
- new net: N41.1, R414.2, R418.1, V406.2 (G)
- new net: C401.1, N40.5 (COMP)
- new net: C401.2, N40.8 (C/B)
- new net: R402.2, V401.2 (C), V405.3 (S)
- new net: R404.1, R405.2
- new net: C415.1, R430.2
- new net +15V: C406.1, C409.1, N40.7 (V+), N41.3 (V+), N42.7 (V+)
- new net +2V5: N41.11 (+), N41.5 (+), N41.7 (+), N41.9 (+)
- new net +5V: C408.2, D40.14 (VDD), D41.16 (VCC), R410.1, R420.1
- new net -15V: C407.1, C410.1, C414.2, N40.4 (V-), N41.12 (V-), N42.4 (V-)
- new net CLK: D40.8 (STB2), D41.3 (CP)
- new net FRQ RG1: R425.1, R426.1, V410.2 (G)
- new net FRQ RG2: R423.1, R424.1, V409.2 (G)
- new net FRQ RG3: R421.1, R422.1, V408.2 (G)
- new net GNDD: C406.2, C407.2, C408.1, C409.2, C410.2, C414.1, C415.2, D40.12 (DGND), D40.2 (IOUT2), D40.3 (AGND), D41.8 (GND), N40.3 (+), N42.3 (+), R411.2, R416.2, R417.2, R418.2, R419.2, R421.2, R423.2, R425.2, R427.2, R428.2, R429.2, V400.3 (E), V401.3 (E), V402.3 (E), V403.3 (E)
- new net LOOP: D40.15 (VREF), R400.1, R401.1, R402.1, R403.1, R405.1, R406.1, R407.1
- new net SD1: D40.7 (SRI)
- new net SIN: C2.1, C402.1, C404.1, C405.1, N42.6, R430.1
- new net WR: D41.1 (STR)
- new net ~{WR}: D40.9 (~{LD2})
Other:
- note added: "-15V TO N31.12 SHEET 03"
- note added: "SHEET 2/3"
- note added: "SHEET 2/3/5"
- note added: "SHEET 2/3/6"
- note added: "SHEET 3"
- note added: "SHEET 3/5"
