File: Schematic/UPL-B1/UPL-B1.kicad_sch (KiCad schematic)
At the start: 0 parts

Commit message: Added Todo on Root page
Other:
- note added: "TODO -Digital Ground vs Analog ground? Today everything is using digital ground. ==> How was the B5 configured? -Finish hierarchical layout on Root page and double check all in and outputs -Start checking all components for availability"
Changed lines of the file:
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@@
 		(company "BVKSound")
+	)
+	(text "TODO\n-Digital Ground vs Analog ground? Today everything is using digital ground.\n==> How was the B5 configured?\n-Finish hierarchical layout on Root page and double check all in and outputs\n-Start checking all components for availability\n"
+		(exclude_from_sim no)
+		(at 199.136 312.674 0)
+		(effects
+			(font
+				(size 5.08 5.08)
+				(thickness 1.016)
+				(bold yes)
+			)
+			(justify left)
+		)
 	)
 	(image

Commit message: Minor fixups for layout.
Reannotate, deduplicate N53B. Add some hierachical pins. First
preparations for layout
Other:
- sheet Integrator 1 & Loop Inverter ports: added ALC, CLK, COS, FRQ_RG1, FRQ_RG2, FRQ_RG3, LOOP, SD1, SD2, SIN, /WR; removed none
- sheet Integrator 2 ports: added CLK, FRQ_RG2, FRQ_RG3, LOOP, SD1, SIN, WR, /WR; removed none
- sheet Output IMD Attenuator ports: added CLK, COS, ENABLE, FILT, FREQ_ENA, LOFILT, LOW DIST, SD2, SDI, SDO, WR, ~{RD}, ~{WR}; removed none

Commit message: Begin redrawing overview page.
Having a huge bitmap in the background makes KiCad lag significantly, so
try to get rid of it.
Other:
- sheet Level Control (ALC) ports: added ALC, COS, FILT, FREQ_ENA, LOFILT, LOFREQ, SIN; removed none
- sheet Output IMD Attenuator ports: added none; removed SDI
- note added: "Integrator 2"
- note added: "N301"
- note added: "N401"

Commit message: Redraw block diagram as vector art. Add more links in hierarchical overview.
Remove original picture
Other:
- sheet Integrator 2 ports: added FRQ_RG1; removed none
- note added: "+ -"
- note added: "-6V2"
- note added: "10Hz ... 110kHz"
- note added: "12bit"
- note added: "COS"
- note added: "D22,N20"
- note added: "D32, N35"
- note added: "D50"
- note added: "D51 N56"
- note added: "DATA LINK"
- note added: "FIXME: SD1 actually is an _INPUT_ on both sides"
- note added: "FREQ TUNE"
- note added: "IMD ATTEN"
- note added: "INTEGRATOR 1"
- note added: "LEVEL CONTROL (ALC)"
- note added: "LOOP INVERTER"
- note added: "N51"
- note added: "N52"
- note added: "N54 V512"
- note added: "REGLER STABILIZER"
- note added: "SUMMIERVERSTÄRKER"
- note added: "SUMMIERVERSTÄRKER SUMMING AMPLIFIER"
- note added: "SUMMING AMPLIFIFER"
- note added: "T & H CONTROL"
- note added: "V500"
- note added: "V5005..V508"
- note added: "V504 C504 N53"
- note added: "V510 C551 N55"
- note added: "V=0..-20dB"
- note added: "V=1,0...0,0"
- note added: "X1A 16"
- note added: "~ 2V7_{EFF}"

Commit message: Clean up overview some more
Other:
- note added: "V505..V508"
- note removed: "V5005..V508"

Commit message: Group functional blocks in ALC. Begin documenting digital chain.
Fixed D21 designator, placed a few NC-Crosses on unused pins for good
practice.
Other:
- sheet Integrator 1 & Loop Inverter ports: added WR, ~{WR}; removed none
- sheet Integrator 2 ports: added ~{WR}; removed /WR
- sheet Output IMD Attenuator ports: added IN_CLK, IN_SDI, SDI, ~{IN_RD}, ~{IN_WR}; removed none
- note removed: "DATA LINK"

Commit message: Rework digital signal chain
Other:
- sheet Output IMD Attenuator ports: added SD1; removed IN_SDI
- note added: "D21"
- note added: "D22"
- note added: "D23"
- note added: "D30"
- note added: "D31"
- note added: "D32"
- note added: "T & H (Track & Hold == Sample & Hold) CONTROL"
- note removed: "FIXME: SD1 actually is an _INPUT_ on both sides"
- note removed: "T & H CONTROL"
