File: Schematic/UPL-B1/Sheet3.kicad_sch (KiCad schematic)
At the start: 103 parts, among them P30 TestPoint, P31 TestPoint, P32 TestPoint, P33 TestPoint, P34 TestPoint

Commit message: ERC fixes.
- Power flags added for power nets "hanging" off resistors.
- Add missing NC-markers for intentionally unconnected parts
- Fix -15V bridge between circuits on S4/S3
- Add +5 to /CLR of DAC
- Use non-hierachical labels on main sheet.
Connections:
- net -15V: no longer C322.2, N31.12 (V-), R348.1
- net ~{WR} renamed /WR
- new net -VDC: C322.2, N31.12 (V-), R348.1
- no-connect marks 1 -> 6
Other:
- moved on the sheet: C315, N33E, R344
