File: Schematic/UPL-B1/Sheet3.kicad_sch (KiCad schematic)
At the start: 103 parts, among them P30 TestPoint, P31 TestPoint, P32 TestPoint, P33 TestPoint, P34 TestPoint

Commit message: Use +/-15VA for some opamps and +5VA for the DACs.
Note: Did they really use +/-15VA (denoted with asterisk in R&S
schematics) on N34 but not on N20?
Connections:
- net +15V: no longer C313.1, N34.7 (V+)
- net +5V: no longer D30.14 (VDD), D32.14 (VDD), R310.1, R341.1
- net -15V: no longer C314.1, N34.4 (V-)
- new net +15VA: C313.1, N34.7 (V+)
- new net +5VA: D30.14 (VDD), D32.14 (VDD), R310.1, R341.1
- new net -15VA: C314.1, N34.4 (V-)
