File: Schematic/UPL-B1/Sheet5.kicad_sch (KiCad schematic)
At the start: 102 parts, among them P53 TestPoint, P54 TestPoint, P55 TestPoint, P56 TestPoint, P57 TestPoint, P58 TestPoint, X50 Conn_01x03_Pin_Bridge, X51 Conn_01x03_Pin_Bridge, X52 Conn_01x03_Pin_Bridge

Commit message: Minor readability changes
Connections:
- net LOFREQ renamed LDFREQ
Changed lines of the file:
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@@
 		)
 	)
-	(hierarchical_label "LOFREQ"
+	(hierarchical_label "LDFREQ"
 		(shape output)
 		(at 317.5 283.21 0)
