File: Schematic/UPL-B1/Integrator 1 & Loop Inverter.kicad_sch (KiCad schematic)
At the start: 103 parts, among them P30 TestPoint, P31 TestPoint, P32 TestPoint, P33 TestPoint, P34 TestPoint

Commit message: Fix wiring of D32
Connections:
- net at C311.1, D32.1 (IOUT1), N35.2 (-)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: now also C311.2, D32.16 (RFB)
Changed lines of the file:
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@@
 	)
 	(junction
+		(at 544.83 223.52)
+		(diameter 0)
+		(color 0 0 0 0)
+	)
+	(junction
 		(at 544.83 160.02)
 		(diameter 0)
@@
 	)
 	(junction
+		(at 482.6 231.14)
+		(diameter 0)
+		(color 0 0 0 0)
+	)
+	(junction
 		(at 142.24 290.83)
 		(diameter 0)
@@
 	(wire
 		(pts
-			(xy 495.3 187.96) (xy 495.3 223.52)
-		)
-		(stroke
-			(width 0)
-			(type default)
-		)
-	)
-	(wire
-		(pts
 			(xy 292.1 293.37) (xy 251.46 293.37)
 		)
@@
 	(wire
 		(pts
+			(xy 495.3 201.93) (xy 544.83 201.93)
+		)
+		(stroke
+			(width 0)
+			(type default)
+		)
+	)
+	(wire
+		(pts
 			(xy 43.18 242.57) (xy 43.18 252.73)
 		)
@@
 	(wire
 		(pts
+			(xy 544.83 201.93) (xy 544.83 223.52)
+		)
+		(stroke
+			(width 0)
+			(type default)
+		)
+	)
+	(wire
+		(pts
 			(xy 392.43 367.03) (xy 389.89 367.03)
 		)
@@
 	(wire
 		(pts
-			(xy 495.3 223.52) (xy 544.83 223.52)
-		)
-		(stroke
-			(width 0)
-			(type default)
-		)
-	)
-	(wire
-		(pts
 			(xy 59.69 87.63) (xy 69.85 87.63)
 		)
@@
 	(wire
 		(pts
+			(xy 482.6 223.52) (xy 544.83 223.52)
+		)
+		(stroke
+			(width 0)
+			(type default)
+		)
+	)
+	(wire
+		(pts
 			(xy 133.35 326.39) (xy 220.98 326.39)
 		)
@@
 	(wire
 		(pts
+			(xy 482.6 231.14) (xy 482.6 223.52)
+		)
+		(stroke
+			(width 0)
+			(type default)
+		)
+	)
+	(wire
+		(pts
 			(xy 233.68 267.97) (xy 229.87 267.97)
 		)
@@
 		)
 		(stroke
+			(width 0)
+			(type default)
+		)
+	)
+	(wire
+		(pts
+			(xy 495.3 187.96) (xy 495.3 201.93)
+		)
+		(stroke

Commit message: Some visual cleanup
Other:
- moved on the sheet: C309, R339
Changed lines of the file:
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@@
 	)
 	(junction
-		(at 495.3 120.65)
-		(diameter 0)
-		(color 0 0 0 0)
-	)
-	(junction
 		(at 156.21 198.12)
 		(diameter 0)
@@
 	)
 	(junction
+		(at 495.3 120.65)
+		(diameter 0)
+		(color 0 0 0 0)
+	)
+	(junction
 		(at 142.24 290.83)
 		(diameter 0)
@@
 	(wire
 		(pts
-			(xy 511.81 132.08) (xy 544.83 132.08)
+			(xy 527.05 132.08) (xy 544.83 132.08)
 		)
 		(stroke
@@
 	(wire
 		(pts
-			(xy 495.3 120.65) (xy 529.59 120.65)
+			(xy 495.3 120.65) (xy 521.97 120.65)
 		)
 		(stroke
@@
 	(wire
 		(pts
-			(xy 534.67 120.65) (xy 544.83 120.65)
+			(xy 527.05 120.65) (xy 544.83 120.65)
 		)
 		(stroke
@@
 	(wire
 		(pts
-			(xy 495.3 132.08) (xy 506.73 132.08)
+			(xy 495.3 132.08) (xy 521.97 132.08)
 		)
 		(stroke
@@
 	(symbol
 		(lib_id "Device:R_Small")
-		(at 509.27 132.08 270)
+		(at 524.51 132.08 270)
 		(mirror x)
 		(unit 1)
@@
 		(dnp no)
 		(property "Reference" "R339"
-			(at 510.286 125.222 90)
+			(at 525.526 125.222 90)
 			(show_name no)
 			(do_not_autoplace no)
@@
 		)
 		(property "Value" "4K75 0.1%"
-			(at 510.286 127.762 90)
+			(at 525.526 127.762 90)
 			(show_name no)
 			(do_not_autoplace no)
@@
 		)
 		(property "Footprint" "R_Axial_DIN0204_L3.6mm_D1.6mm_P7.62mm_Horizontal"
-			(at 509.27 132.08 0)
+			(at 524.51 132.08 0)
 			(hide yes)
 			(show_name no)
@@
 		)
 		(property "Datasheet" ""
-			(at 509.27 132.08 0)
+			(at 524.51 132.08 0)
 			(hide yes)
 			(show_name no)
@@
 		)
 		(property "Description" "Resistor, small symbol"
-			(at 509.27 132.08 0)
+			(at 524.51 132.08 0)
 			(hide yes)
 			(show_name no)
@@
 	(symbol
 		(lib_id "Device:C_Small")
-		(at 532.13 120.65 270)
+		(at 524.51 120.65 270)
 		(unit 1)
 		(body_style 1)
@@
 		(dnp no)
 		(property "Reference" "C309"
-			(at 532.13 114.046 90)
+			(at 524.51 114.046 90)
 			(show_name no)
 			(do_not_autoplace no)
@@
 		)
 		(property "Value" "3p9F"
-			(at 532.13 116.586 90)
+			(at 524.51 116.586 90)
 			(show_name no)
 			(do_not_autoplace no)
@@
 		)
 		(property "Footprint" "Capacitor_SMD:C_1206_3216Metric_Pad1.33x1.80mm_HandSolder"
-			(at 532.13 120.65 0)
+			(at 524.51 120.65 0)
 			(hide yes)
 			(show_name no)
@@
 		)
 		(property "Datasheet" ""
-			(at 532.13 120.65 0)
+			(at 524.51 120.65 0)
 			(hide yes)
 			(show_name no)
@@
 		)
 		(property "Description" "Unpolarized capacitor, small symbol"
-			(at 532.13 120.65 0)
+			(at 524.51 120.65 0)
 			(hide yes)
 			(show_name no)
