File: Schematic/UPL-B1/Level Control (ALC).kicad_sch (KiCad schematic)
At the start: 102 parts, among them P53 TestPoint, P54 TestPoint, P55 TestPoint, P56 TestPoint, P57 TestPoint, P58 TestPoint, X50 Conn_01x03_Pin_Bridge, X51 Conn_01x03_Pin_Bridge, X52 Conn_01x03_Pin_Bridge

Commit message: Some visual cleanup
Other:
- note added: "Is Drain/Source wired up correctly on V504/V510/V512?"
Changed lines of the file:
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@@
 	)
 	(rectangle
-		(start 327.66 115.062)
-		(end 399.542 161.798)
+		(start 327.66 109.982)
+		(end 399.542 199.39)
 		(stroke
 			(width 0)
@@
 	(text "Regler\nStabilizer"
 		(exclude_from_sim no)
-		(at 364.744 112.268 0)
+		(at 364.236 106.934 0)
 		(effects
 			(font
@@
 			)
 		)
+	)
+	(text "Is Drain/Source wired up correctly on V504/V510/V512?"
+		(exclude_from_sim no)
+		(at 246.126 116.84 0)
+		(effects
+			(font
+				(size 1.27 1.27)
+				(color 255 0 43 1)
+			)
+		)

Commit message: Add annotation for glitch in ALC.
The ALC circuit glitches slightly once per sampling. This is not much of
a deal, as this occurs around the zero-value of the sine therefore we do
not expect it to matter regarding sine THD+N.
Other:
- note added: "Expected Waveforms"
- note added: "P53: range=0 gain=2^{11} coarse=0 tune=2^{11}"
- note added: "P58: range=0 gain=2^{11} coarse=0 tune=2^{11}"

Commit message: Remove a bridge that disables C500, C520
Connections:
- net at C500.1, C501.1, C502.2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: no longer C500.2, C520.1, R538.2
- new net: C500.2, C520.1, R538.2
Changed lines of the file:
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@@
 	)
 	(junction
-		(at 82.55 148.59)
-		(diameter 0)
-		(color 0 0 0 0)
-	)
-	(junction
 		(at 113.03 243.84)
 		(diameter 0)
@@
 		)
 	)
-	(wire
-		(pts
-			(xy 82.55 148.59) (xy 92.71 148.59)
-		)
-		(stroke
-			(width 0)
-			(type default)
-		)
-	)
 	(polyline
 		(pts
@@
 		)
 	)
-	(wire
-		(pts
-			(xy 82.55 148.59) (xy 82.55 162.56)
-		)
-		(stroke
-			(width 0)
-			(type default)
-		)
-	)
 	(polyline
 		(pts
@@
 	(wire
 		(pts
-			(xy 78.74 148.59) (xy 82.55 148.59)
+			(xy 78.74 148.59) (xy 92.71 148.59)
 		)
 		(stroke

Commit message: Add more expected waveforms
Other:
- note added: "1/(2*f)"
- note added: "12µs"
- note added: "P30 SIN"
- note added: "P54"
- note added: "P56"
- note added: "P57"
